File: magic_sensor_pcb.kicad_pcb (KiCad board)
At the start: 2 copper layers, 0 parts

Commit message: prepared layout
Parts:
- added C1: 22uF, Capacitor_SMD:C_0603_1608Metric, F.Cu at (65.2, 53.0)
- added C2: 0.1uF, Capacitor_SMD:C_0603_1608Metric, F.Cu at (53.5, 51.0)
- added C3: 0.1uF, Capacitor_SMD:C_0603_1608Metric, F.Cu at (51.0, 53.5)
- added C4: 1uF, Capacitor_SMD:C_0603_1608Metric, F.Cu at (52.0, 64.8)
- added C5: 1uF, Capacitor_SMD:C_0603_1608Metric, F.Cu at (56.5, 66.2)
- added J1: APDS-9960_INT, Connector_PinSocket_2.54mm:PinSocket_1x01_P2.54mm_Vertical, F.Cu at (52.0, 61.0)
- added J2: power, Connector_PinSocket_2.54mm:PinSocket_1x02_P2.54mm_Vertical, F.Cu at (68.0, 52.0)
- added J3: data, Connector_PinSocket_2.54mm:PinSocket_1x02_P2.54mm_Vertical, F.Cu at (68.0, 58.0)
- added R1: 22R, Resistor_SMD:R_0603_1608Metric, F.Cu at (55.5, 63.8)
- added R2: 10k, Resistor_SMD:R_0603_1608Metric, F.Cu at (55.8, 56.5)
- added R3: 10k, Resistor_SMD:R_0603_1608Metric, F.Cu at (56.8, 54.0)
- added U1: BME680, Package_LGA:Bosch_LGA-8_3x3mm_P0.8mm_ClockwisePinNumbering, F.Cu at (53.8, 53.8)
- added U2: APDS-9960, Package_DFN_QFN:DFN-8_2x2mm_P0.5mm, F.Cu at (61.0, 58.0)
Other:
- board outline added: 20 x 15 mm
