File: magic_sensor_pcb.sch (KiCad schematic (older format))
At the start: 0 parts

Commit message: design circuit
Parts:
- added C1: 22uF, Capacitor_SMD:C_0603_1608Metric, symbol Device:C
- added C2, C3: 0.1uF, Capacitor_SMD:C_0603_1608Metric, symbol Device:C
- added C4, C5: 1uF, Capacitor_SMD:C_0603_1608Metric, symbol Device:C
- added J1: APDS-9960_INT, Connector_PinSocket_2.54mm:PinSocket_1x01_P2.54mm_Vertical, symbol Connector_Generic:Conn_01x01
- added J2: power, Connector_PinSocket_2.54mm:PinSocket_1x02_P2.54mm_Vertical, symbol Connector_Generic:Conn_01x02
- added J3: data, Connector_PinSocket_2.54mm:PinSocket_1x02_P2.54mm_Vertical, symbol Connector_Generic:Conn_01x02
- added R1: 22R, Resistor_SMD:R_0603_1608Metric, symbol Device:R
- added R2, R3: 10k, Resistor_SMD:R_0603_1608Metric, symbol Device:R
- added U1: BME680, Package_LGA:Bosch_LGA-8_3x3mm_P0.8mm_ClockwisePinNumbering, symbol Sensor:BME680
- added U2: APDS-9960, OptoDevice:Broadcom_APDS-9960, symbol Sensor_Optical:APDS-9960
Connections:
- new net: J1.1 (Pin_1), U2.2 (INT)
- new net: U2.3 (LDR), U2.4 (LEDK)
- new net +3V3: C1.1, C2.1, C3.1, C4.1, J2.2 (Pin_2), R1.2, R2.1, R3.1, U1.2 (CSB), U1.5 (SDO), U1.6 (VDDIO), U1.8 (VDD), U2.5 (LEDA)
- new net 3.3V_filtered: C5.1, R1.1, U2.8 (VDD)
- new net GND: C1.2, C2.2, C3.2, C4.2, C5.2, J2.1 (Pin_1), U1.1 (GND), U1.7 (GND), U2.6 (GND)
- new net SCL: J3.1 (Pin_1), R2.2, U1.4 (SCK), U2.7 (SCL)
- new net SDA: J3.2 (Pin_2), R3.2, U1.3 (SDI), U2.1 (SDA)
Other:
- note added: "I2C address: 0x39"
- note added: "I2C address: 0x77\nSDO→GND 0x76\nSDO→VDD 0x77"
- note added: "enable I2C mode"
- note added: "supply filtering because \nof High-LED-Currents\nsee Datasheet page34"

Commit message: prepared layout
Parts:
- U2: footprint OptoDevice:Broadcom_APDS-9960 -> Package_DFN_QFN:DFN-8_2x2mm_P0.5mm
Changed lines of the file:
@@
 F 0 "U2" H 5650 4650 50  0000 L CNN
 F 1 "APDS-9960" H 5600 3950 50  0000 L CNN
-F 2 "OptoDevice:Broadcom_APDS-9960" H 5550 4750 50  0001 C CNN
+F 2 "Package_DFN_QFN:DFN-8_2x2mm_P0.5mm" H 5550 4750 50  0001 C CNN
 F 3 "https://docs.broadcom.com/docs/AV02-2315EN" H 5250 4650 50  0001 C CNN
 	1    5550 4300
